File: power-supply/boosst_new.sch (EAGLE design)
At the start: 14 parts

Commit message: slow progress
added new version for in4 PCB + some cleaning of files
Parts:
- removed SL1: (no value), con-amp-quick:M04
- added JP1, JP2: (no value), SparkFun-Connectors:M022.54MM_SCREWTERM
Connections:
- net GND: now also JP1.2, JP2.1; no longer SL1.2, SL1.3
- net VIN: now also JP2.2; no longer SL1.4
- net VOUT: now also JP1.1; no longer SL1.1
