File: nixie-tubes/in4_single_v0.2_revB.brd (EAGLE design)
At the start: 36.8 x 40.6 mm, 17 parts, among them IC1 74HC595D, IC2 74HC595D, IC3 ULN2003AD, IC4 ULN2003AD

Commit message: cleanup, schematic, footprint change
Parts:
- IC1, IC2: device SparkFun-DigitalIC:SO16 -> 74xx-eu:SO16
- R4: device resistor:R1206 -> resistor:R1210
Routing:
- net GND: track 1.40 -> 0.00 mm
- net +5V: track 66.0 -> 67.3 mm
- net CLEAR: track 20.8 -> 21.4 mm
- net LATCH: track 61.9 -> 62.5 mm
- net CLK: track 62.3 -> 62.8 mm
- net N$1: track 34.5 -> 34.0 mm
Other:
- board text added: "IN4 NIXIE v0.2 rev B"
- board text removed: "IN4 NIXIE v0.2 rev A"
